File: demos/git_revision_test/git_revision_test.kicad_sch (KiCad schematic)
At the start: 0 parts

Commit message: Update git revision test project files
Other:
- company: (none) -> GIT REV SHORT ${GIT_REV_SHORT}
Changed lines of the file:
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@@
 	(title_block
 		(rev "${GIT_REV_SHORT}")
+		(company "GIT REV SHORT ${GIT_REV_SHORT}")
 		(comment 1 "GIT REVISION: ${GIT_REVISION}")
 		(comment 2 "GIT TAG: ${GIT_TAG}")
-		(comment 3 "GIT REV SHORT: ${GIT_REV_SHORT}")
+		(comment 3 "VCSHASH: ${VCSHASH}")
+		(comment 4 "VCSSHORTHASH: ${VCSSHORTHASH}")
 	)
 	(sheet_instances
